File: EFUSE2024/EFUSE2024.kicad_sch (KiCad schematic)
At the start: 1 part

Commit message: test
Connections:
- net HIIII_NITYA WAZ_HERE: now also C1.2
Changed lines of the file:
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@@
 	(generator_version "8.0")
 	(paper "A4")
+	(junction
+		(at 69.85 72.39)
+		(diameter 0)
+		(color 0 0 0 0)
+	)
 	(wire
 		(pts
@@
 	(wire
 		(pts
-			(xy 68.58 72.39) (xy 100.33 72.39)
+			(xy 68.58 72.39) (xy 69.85 72.39)
 		)
 		(stroke
+			(width 0)
+			(type default)
+		)
+	)
+	(wire
+		(pts
+			(xy 69.85 72.39) (xy 100.33 72.39)
+		)
+		(stroke
+			(width 0)
+			(type default)
+		)
+	)
+	(wire
+		(pts
+			(xy 69.85 68.58) (xy 68.58 68.58)
+		)
+		(stroke
+			(width 0)
+			(type default)
+		)
+	)
+	(wire
+		(pts
+			(xy 69.85 72.39) (xy 69.85 68.58)
+		)
+		(stroke
